File: Design/P00R1.sch (EAGLE design)
At the start: 2 parts, among them P1 PENTABIT_17.32

Commit message: -Fix some Schematic issues
Other:
- note added: "P00R1_Frontend"
- note removed: "P00R1_Backend"
Changed lines of the file:
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@@
 <text x="180.9242" y="19.6342" size="1.9304" layer="102" font="vector">P00R1</text>
 <text x="191.9478" y="11.2014" size="1.9304" layer="101" font="vector" align="center">Mounting Hole</text>
-<text x="206.3242" y="19.6342" size="1.9304" layer="101" font="vector">P00R1_Backend</text>
+<text x="206.3242" y="19.6342" size="1.9304" layer="101" font="vector">P00R1_Frontend</text>
 <wire x1="168.91" y1="3.81" x2="168.91" y2="8.128" width="0.1524" layer="205"/>
 <wire x1="168.91" y1="8.128" x2="168.91" y2="18.288" width="0.1524" layer="205"/>
